File: sugar-rocket.sch (KiCad schematic (older format))
At the start: 18 parts

Commit message: Made rocket igniter sch
Parts:
- removed J?: Screw_Terminal_01x02, symbol Connector:Screw_Terminal_01x02
- removed J?: Screw_Terminal_01x03, symbol Connector:Screw_Terminal_01x03
- added J1: Conn_01x02, Connector:Banana_Jack_2Pin, symbol Connector_Generic:Conn_01x02
- added J2: Conn_01x03, Connector:Banana_Jack_3Pin, symbol Connector_Generic:Conn_01x03
- D1: renamed from D?; footprint (none) -> Diode_SMD:D_SOD-128
- D2, D3, D5: renamed from D?; footprint (none) -> LED_THT:LED_D5.0mm
- D4, D6: renamed from D?; footprint (none) -> Diode_THT:D_DO-35_SOD27_P5.08mm_Vertical_KathodeUp
- R1, R2, R3: renamed from R?; value R -> 1k; footprint (none) -> Resistor_SMD:R_0805_2012Metric_Pad1.20x1.40mm_HandSolder
- R4, R5: renamed from R?; value R -> 10k; footprint (none) -> Resistor_SMD:R_0805_2012Metric_Pad1.20x1.40mm_HandSolder
- SW1: renamed from SW?; footprint (none) -> Button_Switch_SMD:SW_DPDT_CK_JS202011JCQN
- SW2: renamed from SW?; footprint (none) -> Button_Switch_SMD:SW_Push_1P1T_NO_6x6mm_H9.5mm
- gave numbers to parts that had none: 2
